Commit message: camera rotacionada e aspect ratio 16:9

File: myur5_description/urdf/camera.xacro (robot description, xacro)
@@ -5,5 +5,6 @@
         <parent link="wrist_3_link"/>
         <child link="camera_link"/>
-        <origin xyz="0 0 0" rpy="0 ${-pi/2} ${-pi/2}"/>
+        <origin xyz="0 0 0" rpy="0 ${-pi/2} ${pi}"/>
+        <!-- Rotacionar Camera aqui -->
     </joint>
     <link name="camera_link">
@@ -29,6 +30,6 @@
               <horizontal_fov>1.3962634</horizontal_fov>
               <image>
-                <width>800</width>
-                <height>800</height>
+                <width>1280</width>
+                <height>720</height>
                 <format>R8G8B8</format>
               </image>
